File: Hardware/Kicad/C816SX/C816SX.kicad_pcb (KiCad board)
At the start: 6 copper layers, 99.9 x 99.9 mm, 152 parts, among them IC4 IS61WV20488FBLL-10TLI, J1 Conn_02x06_Odd_Even, J10 5749265-1, J11 Conn_02x06_Odd_Even, J14 Conn_02x03_Odd_Even, J15 Conn_02x03_Odd_Even, J16 Conn_01x06_Pin, J17 Conn_01x09, J18 USB_B, J19 Conn_02x03_Odd_Even, J2 HDMI_A, J20 Conn_02x03_Odd_Even, J21 SD_Card_Receptacle, J22 Conn_01x07_Pin, J23 Conn_01x07_Pin, J25 Conn_01x02, J26 NYS354, J27 NYS354, J4 USB_A_Stacked, J5 DE9_Pins, J9 DE9_Pins, SW1 SW_DIP_x04, U1 W65C816SxQ, U14 W25Q128JVS, U15 SN74LVC8T245PWR, U17 SN74LVC8T245PWR, U18 SN74LVC8T245PWR, U19 SN74LVC8T245PWR, U2 PCM5102A, U20 SN74LVC8T245PWR, U21 SN74LVC8T245PWR, U22 SN74LVC8T245PWR, U3 XC6206PxxxMR, U4 74LVC07, U7 74LVC07, U8 W65C22SxQ, Y2 SiT8008xx-7x-xxE

Commit message: ckeanup
Parts:
- removed R13, R14: 33, Resistor_SMD:R_0805_2012Metric_Pad1.20x1.40mm_HandSolder
- removed R16: 3K3, Resistor_SMD:R_0805_2012Metric_Pad1.20x1.40mm_HandSolder
- removed R21: 1k5, Resistor_SMD:R_0805_2012Metric_Pad1.20x1.40mm_HandSolder
- removed R24: 330, Resistor_SMD:R_0805_2012Metric_Pad1.20x1.40mm_HandSolder
- removed R45: 1K, Resistor_SMD:R_0402_1005Metric
- removed R46, R47: 470, Resistor_SMD:R_0402_1005Metric
- removed R5, R7: 1K, Resistor_SMD:R_0805_2012Metric_Pad1.20x1.40mm_HandSolder
- added C50: 100n, Capacitor_SMD:C_0402_1005Metric, F.Cu at (227.3, 49.5)
- added NT68: NetTie_2, FPGA AND STUFF:MyNetTie-2_SMD_Pad0.25mm, F.Cu at (238.8, 87.3)
- added NT69: NetTie_2, FPGA AND STUFF:MyNetTie-2_SMD_Pad0.25mm, F.Cu at (238.8, 86.7)
- added R27: 330, Resistor_SMD:R_0603_1608Metric, F.Cu at (165.9, 137.1)
- added R28: 1k, Resistor_SMD:R_0603_1608Metric, F.Cu at (246.8, 138.0)
- added R29: 1k, Resistor_SMD:R_0603_1608Metric, F.Cu at (246.8, 136.0)
- added R30: 470, Resistor_SMD:R_0603_1608Metric, F.Cu at (201.5, 51.5)
- added R31: 470, Resistor_SMD:R_0603_1608Metric, F.Cu at (201.5, 53.1)
- added R32: 1k, Resistor_SMD:R_0603_1608Metric, F.Cu at (171.3, 92.7)
- added R34: 1k, Resistor_SMD:R_0603_1608Metric, F.Cu at (224.7, 48.0)
- added R35: 1k5, Resistor_SMD:R_0603_1608Metric, F.Cu at (238.0, 126.8)
- R25, R26: footprint Resistor_SMD:R_0805_2012Metric_Pad1.20x1.40mm_HandSolder -> Resistor_SMD:R_0603_1608Metric
- moved R25 122.3 mm to (182.4, 92.1), turned to 90 degrees
- moved R26 119.1 mm to (185.6, 92.2), turned to 90 degrees
- moved C49 3.63 mm to (226.8, 84.9), turned to 180 degrees
- moved C46 2.11 mm to (199.3, 53.6)
- moved C47 1.64 mm to (199.3, 51.0)
- moved C30 1.29 mm to (208.6, 90.6), turned to 90 degrees
- moved RN6 0.89 mm to (210.1, 93.6)
- moved RN7 0.87 mm to (210.1, 97.7)
- moved Y2 0.37 mm to (229.3, 85.5)
- moved NT54 0.27 mm to (223.3, 59.2)
Routing:
- net GND: track 94.6 -> 131.8 mm, vias 99 -> 110
- net /LVDS_IOR11_N: track 6.70 -> 36.9 mm
- net /ESP_STATUS: track 58.3 -> 37.4 mm
- net /ESP_3V3: track 2.94 -> 21.6 mm
- net /CLKVIA: track 0.00 -> 16.3 mm
- net /_CSVIA: track 0.00 -> 15.8 mm
- net /G14_IOT13B: track 21.7 -> 37.3 mm, vias 2 -> 3
- net /G15_IOT13A: track 21.6 -> 35.5 mm, vias 2 -> 3
- net /ESP_SCL: track 35.4 -> 21.5 mm
- net /RDY.: track 15.4 -> 28.6 mm, vias 2 -> 3
- net /ESP_SDA: track 38.0 -> 27.0 mm
- net +3V3: track 29.5 -> 39.4 mm, vias 25 -> 26
- net Net-(U14-~{HOLD}/~{RESET}/IO_{3}): track 0.00 -> 6.74 mm
- net /LVDS_IOT40_N: track 25.8 -> 19.8 mm, vias 0 -> 2
- net Net-(D1-K): track 0.00 -> 3.50 mm
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