File: Hardware/Kicad/C816SX/C816SX.kicad_sch (KiCad schematic)
At the start: 154 parts, among them IC1 SP720APP, IC2 SP721APP, IC3 SP720APP, J1 Conn_02x20_Odd_Even, J10 5749265-1, J11 Conn_02x06_Odd_Even, J12 Conn_02x12_Odd_Even, J13 Conn_01x03_Pin, J14 Conn_02x03_Odd_Even, J15 Conn_02x03_Odd_Even, J16 Conn_01x06_Pin, J17 Conn_01x09, J18 USB_B, J19 Conn_02x03_Odd_Even, J2 Conn_02x06_Odd_Even, J20 Conn_01x06_Socket, J21 SD_Card_Receptacle, J22 Conn_01x07_Pin, J23 Conn_01x07_Pin, J24 Conn_01x09_Socket, J25 Conn_01x02, J26 NYS354, J27 NYS354, J3 Conn_02x20_Odd_Even, J4 USB_A_Stacked, J5 DE9_Pins, J6 Conn_02x06_Odd_Even, J7 Conn_02x06_Odd_Even, J8 Conn_02x06_Odd_Even, J9 DE9_Pins, SW1 SW_DIP_x04, U1 W65C816SxP, U10 74LVCH245, U11 74LVCH245, U12 74AHCT245, U13 74AHCT245, U14 W25Q128JVS, U2 CY7C1049G-10VXI, U3 CY7C1049G-10VXI, U4 74LVC07, U5 SN74LVC8T245, U6 W65C22NxP, U7 74LVC07, U8 74AHCT245, U9 74LVCH245, Y1 LTC6905xS5-100

Commit message: C816SX
Parts:
- removed C12, C13, C14, C15, C16, C17, C18, C19, C20, C3, C4, C5, C7, C9: 100n, Capacitor_SMD:C_0805_2012Metric_Pad1.18x1.45mm_HandSolder, symbol Device:C
- removed C21: C_Polarized, Capacitor_THT:CP_Radial_D13.0mm_P7.50mm, symbol Device:C_Polarized
- removed D2: D_Zener, Diode_THT:D_5W_P12.70mm_Horizontal, symbol Device:D_Zener
- removed F1: Fuse, Fuse:Fuse_2920_7451Metric, symbol Device:Fuse_Small
- removed F2: Polyfuse, Fuse:Fuse_Bourns_MF-RHT300, symbol Device:Polyfuse
- removed H1, H2, H3, H4: MountingHole, MountingHole:MountingHole_2.5mm, symbol Mechanical:MountingHole
- removed IC1, IC3: SP720APP, Package_DIP:DIP-16_W7.62mm_Socket, symbol PS2:SP720APP
- removed IC2: SP721APP, Package_DIP:DIP-8_W7.62mm_Socket, symbol PS2:SP721APP
- removed J1, J3: Conn_02x20_Odd_Even, Connector_PinHeader_2.54mm:PinHeader_2x20_P2.54mm_Vertical, symbol Connector_Generic:Conn_02x20_Odd_Even
- removed J12: Conn_02x12_Odd_Even, Connector_PinHeader_2.54mm:PinHeader_2x12_P2.54mm_Vertical, symbol Connector_Generic:Conn_02x12_Odd_Even
- removed J13: Conn_01x03_Pin, Jumper:SolderJumper-3_P2.0mm_Open_TrianglePad1.0x1.5mm_NumberLabels, symbol Connector:Conn_01x03_Pin
- removed J2, J6, J7, J8: Conn_02x06_Odd_Even, Connector_PinHeader_2.54mm:PinHeader_2x06_P2.54mm_Vertical, symbol Connector_Generic:Conn_02x06_Odd_Even
- removed J20: Conn_01x06_Socket, Connector_PinHeader_2.54mm:PinHeader_1x06_P2.54mm_Vertical, symbol Connector:Conn_01x06_Socket
- removed J24: Conn_01x09_Socket, Connector_PinHeader_2.54mm:PinHeader_1x09_P2.54mm_Vertical, symbol Connector:Conn_01x09_Socket
- removed R1, R10, R11, R12, R18, R22, R23, R27, R28, R29, R30, R31, R32, R8, R9: 33, Resistor_SMD:R_0805_2012Metric_Pad1.20x1.40mm_HandSolder, symbol Device:R
- removed R17: 1K, Resistor_SMD:R_0805_2012Metric_Pad1.20x1.40mm_HandSolder, symbol Device:R
- removed R19: 330, Resistor_SMD:R_0805_2012Metric_Pad1.20x1.40mm_HandSolder, symbol Device:R
- removed R2: 10K, Resistor_SMD:R_0805_2012Metric_Pad1.20x1.40mm_HandSolder, symbol Device:R
- removed R3: 3k3, Resistor_SMD:R_0805_2012Metric_Pad1.20x1.40mm_HandSolder, symbol Device:R
- removed R34, R4, R6: 3K3, Resistor_SMD:R_0805_2012Metric_Pad1.20x1.40mm_HandSolder, symbol Device:R
- removed RN1, RN2: R_Network10, Resistor_THT:R_Array_SIP11, symbol Device:R_Network10
- removed RN3: R_Network06, Resistor_THT:R_Array_SIP7, symbol Device:R_Network06
- removed U1: W65C816SxP, Package_DIP:DIP-40_W15.24mm, symbol 65XX:W65C816SxP
- removed U10, U11, U9: 74LVCH245, Package_SO:SOIC-20W_7.5x12.8mm_P1.27mm, symbol 74xx:74HC245
- removed U12, U13, U8: 74AHCT245, Package_SO:SOIC-20W_7.5x12.8mm_P1.27mm, symbol 74xx:74HC245
- removed U2, U3: CY7C1049G-10VXI, Package_SO:SOJ-36_10.16x23.495mm_P1.27mm, symbol Memory_RAM:IS61C5128AL-10KLI
- removed U5: SN74LVC8T245, Package_SO:SOIC-24W_7.5x15.4mm_P1.27mm, symbol Logic_LevelTranslator:SN74LVC8T245
- removed U6: W65C22NxP, Package_DIP:DIP-40_W15.24mm, symbol 65XX:W65C22NxP
- removed Y1: LTC6905xS5-100, Package_TO_SOT_SMD:TSOT-23-5, symbol Oscillator:LTC6905xS5-100
- added C22, C23, C24, C25, C26, C27, C28, C29, C30, C31, C32, C33, C34, C35, C36, C37, C38, C39, C40, C41, C42, C43, C44, C45, C48, C49: 100n, Capacitor_SMD:C_0402_1005Metric, symbol Device:C
- added C46, C47: 2.2n, Capacitor_SMD:C_0402_1005Metric, symbol Device:C
- added IC4: IS61WV20488FBLL-10TLI, SOP80P1176X120-44N, symbol PS2:IS61WV20488FBLL-10TLI
- added J1: Conn_02x06_Odd_Even, Connector_PinHeader_2.54mm:PinHeader_2x06_P2.54mm_Vertical, symbol Connector_Generic:Conn_02x06_Odd_Even
- added J2: HDMI_A, Connector_Video:HDMI_A_Molex_208658-1001_Horizontal, symbol Connector:HDMI_A
- added J20: Conn_02x03_Odd_Even, Connector_PinHeader_2.54mm:PinHeader_2x03_P2.54mm_Vertical, symbol Connector_Generic:Conn_02x03_Odd_Even
- added NT67: NetTie_2, FPGA AND STUFF:MyNetTie-2_SMD_Pad0.25mm, symbol Device:NetTie_2
- added R20, R41, R42, R43, R44, R45: 1K, Resistor_SMD:R_0402_1005Metric, symbol Device:R
- added R46, R47: 470, Resistor_SMD:R_0402_1005Metric, symbol Device:R
- added RN10, RN11, RN12, RN18, RN20, RN4, RN6, RN7, RN8, RN9: 33, Resistor_SMD:R_Array_Convex_4x0603, symbol Device:R_Pack04
- added RN13, RN14, RN15, RN16, RN19: 10k, Resistor_SMD:R_Array_Convex_4x0603, symbol Device:R_Pack04
- added RN17: 1k, Resistor_SMD:R_Array_Convex_4x0603, symbol Device:R_Pack04
- added SLOT1: DDR3_204P_SMD, FPGA AND STUFF:DDR3-SMD_0705F0BE40F, symbol Things:DDR3_204P_SMD
- added U1: W65C816SxQ, Package_QFP:LQFP-44_10x10mm_P0.8mm, symbol 65XX:W65C816SxQ
- added U15, U17, U18, U19, U20, U21, U22: SN74LVC8T245PWR, Package_SO:TSSOP-24_4.4x7.8mm_P0.65mm, symbol Fpga:SN74LVC8T245PWR
- added U2: PCM5102A, Package_SO:TSSOP-20_4.4x6.5mm_P0.65mm, symbol Audio:PCM5102A
- added U3: XC6206PxxxMR, Package_TO_SOT_SMD:SOT-23-3, symbol Regulator_Linear:XC6206PxxxMR
- added U8: W65C22SxQ, Package_QFP:LQFP-44_10x10mm_P0.8mm, symbol 65XX:W65C22SxQ
- added Y2: SiT8008xx-7x-xxE, Oscillator:Oscillator_SMD_SiT_PQFN-4Pin_2.0x1.6mm, symbol Oscillator:SiT8008xx-7x-xxE
- C1, C2: value 100n -> 1uF; footprint Capacitor_SMD:C_0805_2012Metric_Pad1.18x1.45mm_HandSolder -> Capacitor_SMD:C_0603_1608Metric
- C10, C11: value 100n -> 10uF; footprint Capacitor_SMD:C_0805_2012Metric_Pad1.18x1.45mm_HandSolder -> Capacitor_SMD:C_0805_2012Metric
- C6, C8: value 100n -> 2.2uF; footprint Capacitor_SMD:C_0805_2012Metric_Pad1.18x1.45mm_HandSolder -> Capacitor_SMD:C_0603_1608Metric
Connections:
- net +3V3: now also C23.1, C25.2, C27.1, C29.1, C30.1, C31.1, C40.1, C41.1, C42.1, C48.1, C49.1, IC4.11 (VDD_1), IC4.33 (VDD_2), J20.6 (Pin_6), RN17.1 (R1.1), RN17.2 (R2.1), SLOT1.22, SLOT1.24, U15.23 (VccB), U15.24 (VccB), U17.23 (VccB), U17.24 (VccB), U18.23 (VccB), U18.24 (VccB), U19.23 (VccB), U19.24 (VccB), U2.1 (CPVDD), U2.20 (DVDD), U20.23 (VccB), U20.24 (VccB), U22.23 (VccB), U22.24 (VccB), Y2.1 (OE), Y2.4 (Vdd)
- net A0: now also U1.4 (A0), U18.4 (A2), U22.17 (B5)
- net A1: now also U1.5 (A1), U18.6 (A4), U22.16 (B6)
- net A10: now also U1.15 (A10), U19.9 (A7)
- net A11: now also U1.16 (A11), U19.10 (A8)
- net A11_IOL15A: now also SLOT1.131
- net A12: now also U1.19 (A12), U18.9 (A7)
- net A12_IOL13B: now also SLOT1.123
- net A13: now also U1.20 (A13), U18.7 (A5)
- net A13_IOR32A_READY: now also IC4.38 (A15), SLOT1.98
- net A14: now also U1.21 (A14), U18.5 (A3)
- net A14_IOL8B: now also SLOT1.113
- net A15: now also U1.22 (A15), U18.3 (A1)
- net A15_IOL2B: now also SLOT1.107
- net A2: now also U1.7 (A2), U18.8 (A6), U22.15 (B7)
- net A3: now also U1.8 (A3), U18.10 (A8), U22.14 (B8)
- net A4: now also U1.9 (A4), U19.3 (A1)
- net A5: now also U1.10 (A5), U19.4 (A2)
- net A6: now also U1.11 (A6), U19.5 (A3)
- net A7: now also U1.12 (A7), U19.6 (A4)
- net A8: now also U1.13 (A8), U19.7 (A5)
- net A9: now also U1.14 (A9), U19.8 (A6)
- net A9_IOL27A: now also SLOT1.148
- net AGND: now also C1.2, C8.2, C43.2, C46.2, C47.2, NT67.2, U2.9 (AGND), U3.1 (GND)
- net A_0: now also IC4.4 (A1), RN6.3 (R3.1)
- net A_1: now also IC4.6 (A3), RN6.1 (R1.1)
- net A_10: now also IC4.26 (A10), RN9.2 (R2.1)
- net A_11: now also IC4.25 (A19), RN9.1 (R1.1)
- net A_12: now also IC4.17 (A6), RN7.2 (R2.1)
- net A_13: now also IC4.7 (A4), RN7.4 (R4.1)
- net A_14: now also IC4.5 (A2), RN6.2 (R2.1)
- net A_15: now also IC4.3 (A0), RN6.4 (R4.1)
- net A_2: now also IC4.16 (A5), RN7.3 (R3.1)
- net A_3: now also IC4.18 (A7), RN7.1 (R1.1)
- net A_4: now also IC4.19 (A8), RN8.4 (R4.1)
- net A_5: now also IC4.20 (A9), RN8.3 (R3.1)
- net A_6: now also IC4.30 (A14), RN8.2 (R2.1)
- net A_7: now also IC4.29 (A13), RN8.1 (R1.1)
- net A_8: now also IC4.28 (A12), RN9.4 (R4.1)
- net A_9: now also IC4.27 (A11), RN9.3 (R3.1)
- net B10_IOR31B_~{RECFG}: now also SLOT1.96
- net B11_IOL13A: now also SLOT1.129
- net B12_IOL7B: now also SLOT1.121
- net B13_IOL8A: now also SLOT1.115
- net B14_IOL2A: now also IC4.40 (A17), SLOT1.109
- net BE: now also RN13.8 (R1.2), U1.34 (BE)
- net BE.: now also RN14.8 (R1.2)
- net C10_IOR39A: now also SLOT1.135
- net C11_IOL15B: now also SLOT1.125
- net C12_IOL7A: now also SLOT1.119
- net C13_IOR32B_DONE: now also SLOT1.136
- net C7_IOL40B_1V5: now also SLOT1.157
- net C9_IOL27B: now also SLOT1.146
- net CA1: now also J20.3 (Pin_3), RN16.8 (R1.2), U8.38 (CA1)
- net CA2: now also J20.4 (Pin_4), RN16.7 (R2.2), U8.37 (CA2)
- net CB1: now also J1.11 (Pin_11), U8.13 (CB1)
- net CB2: now also J1.12 (Pin_12), U8.14 (CB2)
- net CLKVIA: now also U17.15 (B7)
- net CLK_IN: now also SLOT1.81, Y2.3 (OUT)
- net D0: now also U1.30 (D0), U20.3 (A1), U21.21 (B1)
- net D1: now also U1.29 (D1), U20.4 (A2), U21.20 (B2)
- net D10_IOL17A: now also SLOT1.182
- net D11_IOL22A: now also SLOT1.180
- net D2: now also U1.28 (D2), U20.5 (A3), U21.19 (B3)
- net D3: now also U1.27 (D3), U20.6 (A4), U21.18 (B4)
- net D4: now also U1.26 (D4), U20.7 (A5), U21.17 (B5)
- net D5: now also U1.25 (D5), U20.8 (A6), U21.16 (B6)
- net D6: now also U1.24 (D6), U20.9 (A7), U21.15 (B7)
- net D7: now also U1.23 (D7), U20.10 (A8), U21.14 (B8)
- net D7_IOL53B_1V5: now also SLOT1.159
- net DATADIR: now also RN4.8 (R1.2), U20.2 (DIR)
- net DEMP: now also U2.10 (DEMP)
- net E: now also U1.33 (E), U15.9 (A7)
- net E.: now also NT59.1, U15.15 (B7)
- net E10_IOL17B: now also RN17.7 (R2.2), SLOT1.186
- net E8_IOL45B_1V5: now also SLOT1.160
- net E9_IOL38B_1V5: now also SLOT1.158
- net ESP_3V3: now also C22.2
- net F10_IOL11A: now also RN17.8 (R1.2), SLOT1.176
- net F14_IOT9A: now also IC4.13 (I/O2), RN11.2 (R2.1), SLOT1.95
- net F16_IOT9B: now also IC4.14 (I/O3), RN11.1 (R1.1), SLOT1.97
- net FLT: now also U2.11 (FLT)
- net FMT: now also U2.16 (FMT)
- net F_VCCO0&1: now also SLOT1.164, SLOT1.166
- net F_VCCO7: now also SLOT1.170, SLOT1.174
- net G14_IOT13B: now also IC4.32 (I/O5), RN10.2 (R2.1), SLOT1.89
- net G15_IOT13A: now also IC4.31 (I/O4), RN10.1 (R1.1), SLOT1.91
- net GND: now also C22.1, C23.2, C24.1, C25.1, C26.2, C27.2, C28.2, C29.2, C30.2, C31.2, C32.2, C33.2, C34.2, C35.2, C36.2, C37.2, C38.2, C39.2, C40.2, C41.2, C42.2, C44.2, C45.2, C48.2, C49.2, IC4.12 (VSS_1), IC4.34 (VSS_2), J1.2 (Pin_2), J2.11 (CKS), J2.17 (GND), J2.2 (D2S), J2.5 (D1S), J2.8 (D0S), J2.SH, NT67.1, R41.2, RN12.1 (R1.1), RN14.1 (R1.1), SLOT1.127, SLOT1.128, SLOT1.13, SLOT1.133, SLOT1.134, SLOT1.138, SLOT1.139, SLOT1.14, SLOT1.144, SLOT1.145, SLOT1.150, SLOT1.151, SLOT1.155, SLOT1.156, SLOT1.161, SLOT1.162, SLOT1.167, SLOT1.168, SLOT1.172, SLOT1.173, SLOT1.178, SLOT1.179, SLOT1.184, SLOT1.185, SLOT1.189, SLOT1.19, SLOT1.190, SLOT1.195, SLOT1.196, SLOT1.2, SLOT1.20, SLOT1.25, SLOT1.26, SLOT1.3, SLOT1.31, SLOT1.32, SLOT1.37, SLOT1.38, SLOT1.43, SLOT1.48, SLOT1.49, SLOT1.54, SLOT1.55, SLOT1.60, SLOT1.61, SLOT1.66, SLOT1.71, SLOT1.72, SLOT1.8, SLOT1.9, SLOT1.MP, U1.17 (VSS), U1.18 (VSS), U1.39 (VSS), U15.11 (GND), U15.12 (GND), U15.13 (GND), U15.22 (~{OE}), U15.3 (A1), U15.4 (A2), U17.11 (GND), U17.12 (GND), U17.13 (GND), U17.22 (~{OE}), U18.11 (GND), U18.12 (GND), U18.13 (GND), U18.22 (~{OE}), U19.11 (GND), U19.12 (GND), U19.13 (GND), U19.22 (~{OE}), U2.19 (DGND), U2.3 (CPGND), U20.11 (GND), U20.12 (GND), U20.13 (GND), U20.22 (~{OE}), U21.11 (GND), U21.12 (GND), U21.13 (GND), U22.11 (GND), U22.12 (GND), U22.13 (GND), U22.2 (DIR), U22.22 (~{OE}), U8.39 (VSS), Y2.2 (GND); no longer C1.2, C6.2, C8.2
- net I2S_BCK: now also RN12.7 (R2.2), U2.13 (BCK)
- net I2S_DIN: now also RN12.6 (R3.2), U2.14 (DIN)
- net I2S_LRCK: now also RN12.5 (R4.2), U2.15 (LRCK)
- net JTAG_TCK: now also SLOT1.149
- net JTAG_TDI: now also SLOT1.153
- net JTAG_TDO: now also SLOT1.147
- net JTAG_TMS: now also SLOT1.143
- net L: now also J26.1, C47.1, R46.1; no longer J27.1
- net LVDS_IOR11_N: now also IC4.15 (WE#), SLOT1.65, U15.14 (B8)
- net LVDS_IOR11_P: now also SLOT1.63
- net LVDS_IOR17_N: now also RN12.3 (R3.1), SLOT1.59
- net LVDS_IOR17_P: now also RN12.2 (R2.1), SLOT1.57
- net LVDS_IOR20_N: now also SLOT1.69, U17.16 (B6)
- net LVDS_IOR20_P: now also IC4.8 (CS#), SLOT1.67
- net LVDS_IOR24_N: now also SLOT1.51
- net LVDS_IOR24_P: now also SLOT1.53
- net LVDS_IOR29_N: now also J2.6 (D1-), SLOT1.35
- net LVDS_IOR29_P: now also J2.4 (D1+), SLOT1.33
- net LVDS_IOR38_N: now also SLOT1.47
- net LVDS_IOR38_P: now also SLOT1.45
- net LVDS_IOR40_N: now also SLOT1.193
- net LVDS_IOR40_P: now also SLOT1.191
- net LVDS_IOR42_N: now also SLOT1.39
- net LVDS_IOR42_P: now also SLOT1.41
- net LVDS_IOR44_N: now also RN18.1 (R1.1), SLOT1.200
- net LVDS_IOR44_P: now also RN18.2 (R2.1), SLOT1.198
- net LVDS_IOR49_N: now also RN18.3 (R3.1), SLOT1.194
- net LVDS_IOR49_P: now also RN18.4 (R4.1), SLOT1.192
- net LVDS_IOR53_N: now also J2.1 (D2+), SLOT1.27
- net LVDS_IOR53_P: now also J2.3 (D2-), SLOT1.29
- net LVDS_IOT14_N: now also SLOT1.90
- net LVDS_IOT14_P: now also SLOT1.92
- net LVDS_IOT18_N: now also SLOT1.86
- net LVDS_IOT18_P: now also SLOT1.84
- net LVDS_IOT22_N: now also IC4.10 (I/O1), RN11.3 (R3.1), SLOT1.85
- net LVDS_IOT22_P: now also IC4.9 (I/O0), RN11.4 (R4.1), SLOT1.83
- net LVDS_IOT32_N: now also RN20.1 (R1.1), SLOT1.152
- net LVDS_IOT32_P: now also RN20.2 (R2.1), SLOT1.154
- net LVDS_IOT36_N: now also SLOT1.78
- net LVDS_IOT36_P: now also IC4.39 (A16), SLOT1.80
- net LVDS_IOT38_N: now also SLOT1.74
- net LVDS_IOT38_P: now also RN12.4 (R4.1), SLOT1.76
- net LVDS_IOT40_N: now also IC4.37 (OE#), SLOT1.73
- net LVDS_IOT40_P: now also SLOT1.75, U17.14 (B8)
- net LVDS_IOT44_N: now also IC4.42 (A20), SLOT1.101
- net LVDS_IOT44_P: now also IC4.41 (A18), SLOT1.103
- net LVDS_IOT8_N: now also IC4.35 (I/O6), RN10.3 (R3.1), SLOT1.79
- net LVDS_IOT8_P: now also IC4.36 (I/O7), RN10.4 (R4.1), SLOT1.77
- net LVDS_RX1_N: now also SLOT1.50
- net LVDS_RX1_P: now also SLOT1.52
- net LVDS_RX2_N: now also SLOT1.46
- net LVDS_RX2_P: now also SLOT1.44
- net LVDS_RX3_N: now also SLOT1.42
- net LVDS_RX3_P: now also SLOT1.40
- net LVDS_RX4_N: now also J2.9 (D0-), SLOT1.34
- net LVDS_RX4_P: now also J2.7 (D0+), SLOT1.36
- net LVDS_RX5_N: now also J2.12 (CK-), SLOT1.28
- net LVDS_RX5_P: now also J2.10 (CK+), SLOT1.30
- net LVDS_TX1_N: now also SLOT1.142
- net LVDS_TX1_P: now also SLOT1.140
- net LVDS_TX2_N: now also SLOT1.132
- net LVDS_TX2_P: now also SLOT1.130
- net LVDS_TX3_N: now also SLOT1.70
- net LVDS_TX3_P: now also SLOT1.68
- net LVDS_TX4_N: now also SLOT1.62
- net LVDS_TX4_P: now also SLOT1.64
- net LVDS_TX5_N: now also SLOT1.56
- net LVDS_TX5_P: now also SLOT1.58
- net M11_IOR27B_FPGA_TXO: now also SLOT1.11
- net MX: now also U1.36 (MX)
- net N6_IOR51A: now also SLOT1.175
- net N7_IOR47B: now also SLOT1.177
- net N9_IOR36B: now also SLOT1.181
- net PA0: now also J20.1 (Pin_1), RN16.6 (R3.2), U8.40 (PA0)
- net PA1: now also J20.2 (Pin_2), RN16.5 (R4.2), U8.41 (PA1)
- net PA2: now also RN15.7 (R2.2), U8.42 (PA2)
- net PA3: now also RN15.8 (R1.2), U8.43 (PA3)
- net PA4: now also RN19.8 (R1.2), U8.44 (PA4)
- net PA5: now also RN19.7 (R2.2), U8.1 (PA5)
- net PA6: now also RN15.6 (R3.2), U8.2 (PA6)
- net PA7: now also RN15.5 (R4.2), U8.3 (PA7)
- net PB0: now also J1.3 (Pin_3), U8.4 (PB0)
- net PB1: now also J1.4 (Pin_4), U8.6 (PB1)
- net PB2: now also J1.5 (Pin_5), U8.7 (PB2)
- net PB3: now also J1.6 (Pin_6), U8.8 (PB3)
- net PB4: now also J1.7 (Pin_7), U8.9 (PB4)
- net PB5: now also J1.8 (Pin_8), U8.10 (PB5)
- net PB6: now also J1.9 (Pin_9), U8.11 (PB6)
- net PB7: now also J1.10 (Pin_10), U8.12 (PB7)
- net PHI2: now also RN4.6 (R3.2), U1.35 (ϕ0)
- net PHI2.2: now also RN4.7 (R2.2), U8.21 (ϕ2)
- net PS2DAT: now also RN17.5 (R4.2)
- net PSCLK: now also RN17.6 (R3.2)
- net R: now also J27.1, C46.1, R47.1; no longer J26.1
- net R9_IOR35A: now also SLOT1.183
- net RDY: now also R44.2, U1.41 (RDY), U15.5 (A3)
- net RDY.: now also U15.19 (B3), U17.21 (B1)
- net RS0: now also U22.7 (A5), U8.36 (RS0)
- net RS1: now also U22.8 (A6), U8.35 (RS1)
- net RS2: now also U22.9 (A7), U8.34 (RS2)
- net RS3: now also U22.10 (A8), U8.33 (RS3)
- net RW: now also U1.32 (R/~{W}), U15.10 (A8), U22.18 (B4)
- net T10_IOR35B_FPGA_~{RST}: now also SLOT1.15
- net T13_IOR8B_FPGA_RXO: now also SLOT1.1
- net T2_IOB48B_1V5: now also SLOT1.163
- net T3_IOB52B_1V5: now also SLOT1.165
- net T4_IOB45B_1V5: now also SLOT1.169
- net T5_IOB54B_1V5: now also SLOT1.171
- net UD1N: now also RN18.6 (R3.2)
- net UD1P: now also RN18.5 (R4.2)
- net UD2N: now also RN18.8 (R1.2)
- net UD2P: now also RN18.7 (R2.2)
- net UD3N: now also RN20.8 (R1.2)
- net UD3P: now also RN20.6 (R3.2), RN20.7 (R2.2); no longer R21.2
- net VBUS: no longer J10.4, J14.2 (Pin_2), J15.2 (Pin_2), J4.1 (VBUS1), J4.5 (VBUS2)
- net VCC: now also J10.4, J14.2 (Pin_2), J15.2 (Pin_2), J25.2 (Pin_2), J4.1 (VBUS1), J4.5 (VBUS2), C24.2, C26.1, C28.1, C32.1, C33.1, C34.1, C35.1, C36.1, C37.1, C38.1, C39.1, C44.1, J1.1 (Pin_1), J2.18 (+5V), R20.2, R42.2, R43.2, R45.2, RN13.1 (R1.1), RN13.2 (R2.1), RN13.3 (R3.1), RN13.4 (R4.1), RN14.4 (R4.1), RN15.1 (R1.1), RN15.2 (R2.1), RN15.3 (R3.1), RN15.4 (R4.1), RN16.1 (R1.1), RN16.2 (R2.1), RN16.3 (R3.1), RN16.4 (R4.1), RN17.3 (R3.1), RN17.4 (R4.1), RN19.1 (R1.1), RN19.2 (R2.1), RN19.3 (R3.1), RN19.4 (R4.1), SLOT1.4, SLOT1.5, SLOT1.6, SLOT1.7, U1.3 (VDD), U1.31 (VDD), U15.1 (VccA), U17.1 (VccA), U18.1 (VccA), U19.1 (VccA), U20.1 (VccA), U21.1 (VccA), U21.23 (VccB), U21.24 (VccB), U22.1 (VccA), U3.3 (VI), U8.15 (VDD), U8.20 (CS1); no longer C1.1, C10.1, C6.1, C8.1
- net VD0: now also U21.3 (A1), U8.30 (D0)
- net VD1: now also U21.4 (A2), U8.29 (D1)
- net VD2: now also U21.5 (A3), U8.28 (D2)
- net VD3: now also U21.6 (A4), U8.26 (D3)
- net VD4: now also U21.7 (A5), U8.25 (D4)
- net VD5: now also U21.8 (A6), U8.24 (D5)
- net VD6: now also U21.9 (A7), U8.23 (D6)
- net VD7: now also U21.10 (A8), U8.22 (D7)
- net VDA: now also U1.37 (VDA), U15.7 (A5)
- net VDA.: now also NT61.1, U15.17 (B5)
- net VPA: now also U1.2 (VPA), U15.8 (A6)
- net VPA.: now also NT60.1, U15.16 (B6)
- net XSMT: now also U2.17 (XSMT)
- net _ABT: now also RN13.6 (R3.2), U1.42 (~{ABORT})
- net _CS2_VIA: now also RN4.5 (R4.2), U21.22 (~{OE}), U8.19 (~{CS2})
- net _CSVIA: now also U17.17 (B5)
- net _IRQ: now also RN13.7 (R2.2), U1.43 (~{IRQ})
- net _IRQ.2: now also R45.1, U8.17 (~{IRQ})
- net _NMI: now also RN13.5 (R4.2), U1.1 (~{NMI})
- net _RESET: now also RN14.5 (R4.2), U1.38 (~{RES}), U8.31 (~{RES})
- net _RWVIA: now also U22.6 (A4), U8.18 (R/~{W})
- net _VP: now also U1.40 (~{VP}), U15.6 (A4)
- net _VP.: now also NT62.1, U15.18 (B4)
- net _WE: now also U21.2 (DIR)
- net _816: now reaches J17.2 (Pin_2), U4.12
- new net: R47.2, U2.7 (OUTR)
- new net: RN11.8 (R1.2), U20.14 (B8)
- new net: RN11.7 (R2.2), U20.15 (B7)
- new net: RN11.6 (R3.2), U20.16 (B6)
- new net: RN11.5 (R4.2), U20.17 (B5)
- new net: RN10.8 (R1.2), U20.18 (B4)
- new net: RN10.7 (R2.2), U20.19 (B3)
- new net: RN10.6 (R3.2), U20.20 (B2)
- new net: RN10.5 (R4.2), U20.21 (B1)
- new net: RN7.5 (R4.2), U18.17 (B5)
- new net: RN7.6 (R3.2), U18.16 (B6)
- new net: RN7.7 (R2.2), U18.15 (B7)
- new net: RN7.8 (R1.2), U18.14 (B8)
- new net: RN20.3 (R3.1), RN20.4 (R4.1)
- new net: R21.2, RN20.5 (R4.2)
- new net: R42.1, U18.2 (DIR)
- new net: R41.1, U17.2 (DIR)
- new net: RN4.1 (R1.1), U17.10 (A8)
- new net: R44.1, U17.3 (A1)
- new net: RN4.4 (R4.1), U17.7 (A5)
- new net: RN4.3 (R3.1), U17.8 (A6)
- new net: RN4.2 (R2.1), U17.9 (A7)
- new net: RN9.8 (R1.2), U19.14 (B8)
- new net: RN9.7 (R2.2), U19.15 (B7)
- new net: RN9.6 (R3.2), U19.16 (B6)
- new net: RN9.5 (R4.2), U19.17 (B5)
- new net: RN8.8 (R1.2), U19.18 (B4)
- new net: RN8.7 (R2.2), U19.19 (B3)
- new net: R43.1, U19.2 (DIR)
- new net: RN8.6 (R3.2), U19.20 (B2)
- new net: RN8.5 (R4.2), U19.21 (B1)
- new net: C8.1, U2.5 (VNEG)
- new net: R46.2, U2.6 (OUTL)
- new net: RN6.8 (R1.2), U18.18 (B4)
- new net: RN6.7 (R2.2), U18.19 (B3)
- new net: RN6.6 (R3.2), U18.20 (B2)
- new net: RN6.5 (R4.2), U18.21 (B1)
- new net: C6.1, U2.2 (CAPP)
- new net: C6.2, U2.4 (CAPM)
- new net: RN12.8 (R1.2), U2.12 (SCK)
- new net: C10.1, C45.1, U2.18 (LDOO)
- new net: R20.1, U15.2 (DIR)
- new net AVDD: C1.1, C43.1, U2.8 (AVDD), U3.2 (VO)
- new net PULLUP: J20.5 (Pin_5), RN19.5 (R4.2), RN19.6 (R3.2)
- no-connect marks 60 -> 67
Other:
- note added: "A <- B"
- note added: "A <--> B"
- note added: "A->B"
- note added: "A16"
- note added: "A17"
- note added: "A18"
- note added: "A19"
- note added: "A20"
- note added: "AUDIO"
- note added: "B -> A"
- note added: "MEMORY 2048K * 8 10nS ASYNC SRAM"
- note added: "READ VIA B <- A WRITE VIA B -> A"
- note added: "RW."
- note added: "USB SERIAL"
- note added: "_CE1"
- note added: "_RE"
- note removed: "0/IOT6A/E15 or E16"
- note removed: "3/IOR42B/M6 OR P8"
- note removed: "CPU BUS"
- note removed: "IO BUS"
- note removed: "MEMORY 2X 512K * 8 10nS ASYNC SRAM"
- note removed: "MISC"
- note removed: "RW"
- moved on the sheet: J25, R13, R14, U7C, U7D, U7G

Commit message: ckeanup
Parts:
- removed R13, R14: 33, Resistor_SMD:R_0805_2012Metric_Pad1.20x1.40mm_HandSolder, symbol Device:R
- removed R16: 3K3, Resistor_SMD:R_0805_2012Metric_Pad1.20x1.40mm_HandSolder, symbol Device:R
- removed R21: 1k5, Resistor_SMD:R_0805_2012Metric_Pad1.20x1.40mm_HandSolder, symbol Device:R
- removed R24: 330, Resistor_SMD:R_0805_2012Metric_Pad1.20x1.40mm_HandSolder, symbol Device:R
- removed R45: 1K, Resistor_SMD:R_0402_1005Metric, symbol Device:R
- removed R46, R47: 470, Resistor_SMD:R_0402_1005Metric, symbol Device:R
- removed R5, R7: 1K, Resistor_SMD:R_0805_2012Metric_Pad1.20x1.40mm_HandSolder, symbol Device:R
- added C50: 100n, Capacitor_SMD:C_0402_1005Metric, symbol Device:C
- added NT68, NT69: NetTie_2, FPGA AND STUFF:MyNetTie-2_SMD_Pad0.25mm, symbol Device:NetTie_2
- added R27: 330, Resistor_SMD:R_0603_1608Metric, symbol Device:R
- added R28, R29, R32, R34: 1k, Resistor_SMD:R_0603_1608Metric, symbol Device:R
- added R30, R31: 470, Resistor_SMD:R_0603_1608Metric, symbol Device:R
- added R35: 1k5, Resistor_SMD:R_0603_1608Metric, symbol Device:R
- R25, R26: footprint Resistor_SMD:R_0805_2012Metric_Pad1.20x1.40mm_HandSolder -> Resistor_SMD:R_0603_1608Metric
Connections:
- net +3V3: now also C50.1, R28.2, R29.1, R34.1
- net CLKVIA: now also NT68.1
- net E10_IOL17B: now also R28.1
- net F10_IOL11A: now also R29.2
- net GND: now also C50.2, R27.2
- net L: now also R30.1
- net LVDS_IOT14_N: now also NT69.2
- net LVDS_IOT14_P: now also NT68.2
- net R: now also R31.1
- net USB3_CON: now also R35.2
- net VCC: now also R32.1
- net _CSVIA: now also NT69.1
- net _IRQ.2: now also R32.2
- net at U2.7 (OUTR): now also R31.2
- net at RN20.5 (R4.2): now also R35.1
- net at D1.1 (K): now also R27.1
- net at U2.6 (OUTL): now also R30.2
- net at U14.7 (~{HOLD}/~{RESET}/IO_{3}): now also R34.2
- no-connect marks 67 -> 66

Commit message: WIP
Parts:
- removed C10: 10uF, Capacitor_SMD:C_0805_2012Metric, symbol Device:C
- removed C2: 1uF, Capacitor_SMD:C_0603_1608Metric, symbol Device:C
- removed C22, C23, C24, C25, C26, C27, C28, C29, C30, C31, C32, C33, C34, C35, C36, C37, C38, C39, C40, C41, C42, C43, C44, C45, C48, C49, C50: 100n, Capacitor_SMD:C_0402_1005Metric, symbol Device:C
- removed C46, C47: 2.2n, Capacitor_SMD:C_0402_1005Metric, symbol Device:C
- removed C6, C8: 2.2uF, Capacitor_SMD:C_0603_1608Metric, symbol Device:C
- removed D1: LED, LED_THT:LED_D5.0mm_Horizontal_O6.35mm_Z3.0mm, symbol Device:LED
- removed IC4: IS61WV20488FBLL-10TLI, SOP80P1176X120-44N, symbol PS2:IS61WV20488FBLL-10TLI
- removed J14, J15, J19, J20: Conn_02x03_Odd_Even, Connector_PinHeader_2.54mm:PinHeader_2x03_P2.54mm_Vertical, symbol Connector_Generic:Conn_02x03_Odd_Even
- removed J16: Conn_01x06_Pin, Connector_PinSocket_2.54mm:PinSocket_1x06_P2.54mm_Vertical, symbol Connector:Conn_01x06_Pin
- removed J17: Conn_01x09, Connector_PinSocket_2.54mm:PinSocket_1x09_P2.54mm_Vertical, symbol Connector_Generic:Conn_01x09
- removed J18: USB_B, Connector_USB:USB_B_Lumberg_2411_02_Horizontal, symbol Connector:USB_B
- removed J2: HDMI_A, Connector_Video:HDMI_A_Molex_208658-1001_Horizontal, symbol Connector:HDMI_A
- removed J21: SD_Card_Receptacle, Connector_Card:SD_TE_2041021, symbol Connector:SD_Card_Receptacle
- removed J22, J23: Conn_01x07_Pin, Connector_PinSocket_2.54mm:PinSocket_1x07_P2.54mm_Vertical, symbol Connector:Conn_01x07_Pin
- removed J26, J27: NYS354, NYS354, symbol PS2:NYS354
- removed J4: USB_A_Stacked, Connector_USB:USB_A_Wuerth_61400826021_Horizontal_Stacked, symbol Connector:USB_A_Stacked
- removed NT23, NT24, NT25, NT26, NT27, NT28, NT29, NT30, NT31, NT32, NT33, NT34, NT35, NT36, NT37, NT38, NT39, NT40, NT42, NT43, NT44, NT45, NT48, NT51, NT52, NT53, NT54, NT55, NT56, NT57, NT58, NT59, NT60, NT61, NT62, NT63, NT64, NT65, NT66, NT67, NT68, NT69: NetTie_2, FPGA AND STUFF:MyNetTie-2_SMD_Pad0.25mm, symbol Device:NetTie_2
- removed R15: 3K3, Resistor_SMD:R_0805_2012Metric_Pad1.20x1.40mm_HandSolder, symbol Device:R
- removed R20, R41, R42, R43, R44: 1K, Resistor_SMD:R_0402_1005Metric, symbol Device:R
- removed R25, R26, R28, R29, R32, R34: 1k, Resistor_SMD:R_0603_1608Metric, symbol Device:R
- removed R27: 330, Resistor_SMD:R_0603_1608Metric, symbol Device:R
- removed R30, R31: 470, Resistor_SMD:R_0603_1608Metric, symbol Device:R
- removed R33: 330, Resistor_SMD:R_0805_2012Metric_Pad1.20x1.40mm_HandSolder, symbol Device:R
- removed R35: 1k5, Resistor_SMD:R_0603_1608Metric, symbol Device:R
- removed RN12, RN18, RN20: 33, Resistor_SMD:R_Array_Convex_4x0603, symbol Device:R_Pack04
- removed RN14, RN15, RN16, RN19: 10k, Resistor_SMD:R_Array_Convex_4x0603, symbol Device:R_Pack04
- removed SW1: SW_DIP_x04, Button_Switch_THT:SW_DIP_SPSTx04_Piano_10.8x11.72mm_W7.62mm_P2.54mm, symbol Switch:SW_DIP_x04
- removed U2: PCM5102A, Package_SO:TSSOP-20_4.4x6.5mm_P0.65mm, symbol Audio:PCM5102A
- removed U3: XC6206PxxxMR, Package_TO_SOT_SMD:SOT-23-3, symbol Regulator_Linear:XC6206PxxxMR
- added C3: 1000uF, Capacitor_THT:C_Radial_D8.0mm_H7.0mm_P3.50mm, symbol Device:C_Polarized
- added D1: 1N5919BRLG, Diode_THT:D_DO-201_P15.24mm_Horizontal, symbol Diode:1N53xxB
- added F1: Polyfuse_Small, Fuse:Fuse_Littelfuse-LVR200, symbol Device:Polyfuse_Small
- added FID1, FID2, FID3: Fiducial, Fiducial:Fiducial_1mm_Mask2mm, symbol Mechanical:Fiducial
- added J1: Conn_01x08_Pin, Connector_PinHeader_2.54mm:PinHeader_1x08_P2.54mm_Vertical, symbol Connector:Conn_01x08_Pin
- added J3: SD_Card_Receptacle, Connector_Card:SD_TE_2041021, symbol Connector:SD_Card_Receptacle
- added J6: Conn_02x06_Odd_Even, Connector_PinHeader_2.54mm:PinHeader_2x06_P2.54mm_Vertical, symbol Connector_Generic:Conn_02x06_Odd_Even
- added R1, R3, R4: 1k, Resistor_SMD:R_0603_1608Metric, symbol Device:R
- added R2: 470, Resistor_SMD:R_0603_1608Metric, symbol Device:R
- added RN9: 10k, Resistor_SMD:R_Array_Convex_4x0603, symbol Device:R_Pack04
- added SW1: SW_DIP_x02, Button_Switch_THT:SW_DIP_SPSTx02_Slide_9.78x7.26mm_W7.62mm_P2.54mm, symbol Switch:SW_DIP_x02
- added U12: W25Q128JVS, Package_SO:SOIC-8_5.3x5.3mm_P1.27mm, symbol Memory_Flash:W25Q128JVS
- added U24, U25: SP720APP, Package_SO:SOIC-16_3.9x9.9mm_P1.27mm, symbol PS2:SP720APP
- C1: value 1uF -> 2.2uF
- C2: renamed from C11; value 10uF -> 1uF
- renumbered H5 to H1, H6 to H2, H7 to H3, H8 to H4, J11 to J2, J25 to J4, J10 to J5, J1 to J7, J5 to J8, RN8 to RN1, RN17 to RN10, RN9 to RN2, RN4 to RN3, RN6 to RN4, RN7 to RN5, RN10 to RN6, RN11 to RN7, RN13 to RN8, U19 to U1, U8 to U10, U21 to U11, U14 to U13, U17 to U2, U18 to U3, U20 to U4, U1 to U5, U15 to U6, U4 to U7, U7 to U8, U22 to U9, Y2 to Y1
Connections:
- net A11_IOL15A is gone; now on net A_1: SLOT1.131
- net A12_IOL13B is gone; now on net A_4: SLOT1.123
- net A14_IOL8B is gone; now on net A_10: SLOT1.113
- net A15_IOL2B is gone; now on net A_12: SLOT1.107
- net A9_IOL27A is gone; now on net A_6: SLOT1.148
- net AGND is gone; now on net GND: C1.2
- net B11_IOL13A is gone; now on net A_2: SLOT1.129
- net B12_IOL7B is gone; now on net A_5: SLOT1.121
- net B13_IOL8A is gone; now on net A_9: SLOT1.115
- net B14_IOL2A is gone; now on net A_11: SLOT1.109
- net C10_IOR39A is gone; now on net A_0: SLOT1.135
- net C11_IOL15B is gone; now on net A_3: SLOT1.125
- net C12_IOL7A is gone; now on net A_8: SLOT1.119
- net C13_IOR32B_DONE is gone; now on net USB3_CON: SLOT1.136
- net C9_IOL27B is gone; now on net A_7: SLOT1.146
- net LVDS_IOR11_P is gone; now on net I2S_BCK: SLOT1.63
- net LVDS_IOR17_N is gone; now on net I2S_DIN: SLOT1.59
- net LVDS_IOR17_P is gone; now on net I2S_LRCK: SLOT1.57
- net LVDS_IOR24_N is gone; now on net _VP.: SLOT1.51
- net LVDS_IOR24_P is gone; now on net VDA.: SLOT1.53
- net LVDS_IOR29_N is gone; now on net TMDS0_P: SLOT1.35
- net LVDS_IOR29_P is gone; now on net TMDS0_N: SLOT1.33
- net LVDS_IOR38_N is gone; now on net TMDS2_P: SLOT1.47
- net LVDS_IOR38_P is gone; now on net TMDS2_N: SLOT1.45
- net LVDS_IOR40_N is gone; now on net _CESD: SLOT1.193
- net LVDS_IOR42_N is gone; now on net TMDS1_N: SLOT1.39
- net LVDS_IOR42_P is gone; now on net TMDS1_P: SLOT1.41
- net LVDS_IOR44_N is gone; now on net UD2N: SLOT1.200
- net LVDS_IOR44_P is gone; now on net UD2P: SLOT1.198
- net LVDS_IOR49_N is gone; now on net UD1P: SLOT1.194
- net LVDS_IOR49_P is gone; now on net UD1N: SLOT1.192
- net LVDS_IOR53_N is gone; now on net TMDSC_N: SLOT1.27
- net LVDS_IOR53_P is gone; now on net TMDSC_P: SLOT1.29
- net LVDS_IOT14_N is gone; now on net _CSVIA: SLOT1.90
- net LVDS_IOT14_P is gone; now on net CLKVIA: SLOT1.92
- net LVDS_IOT18_N is gone; now on net A_15: SLOT1.86
- net LVDS_IOT40_N is gone; now on net _RE: SLOT1.73
- net LVDS_IOT40_P is gone; now on net DATADIR: SLOT1.75, U2.14 (B8)
- net LVDS_IOT44_N is gone; now on net A_14: SLOT1.101
- net LVDS_IOT44_P is gone; now on net A_13: SLOT1.103
- net LVDS_RX1_N is gone; now on net PS2DATIN: SLOT1.50
- net LVDS_TX1_N is gone; now on net ESP_RX: SLOT1.142
- net LVDS_TX1_P is gone; now on net EPS_CTS: SLOT1.140
- net LVDS_TX2_N is gone; now on net ESP_RTS: SLOT1.132
- net LVDS_TX2_P is gone; now on net ESP_TX: SLOT1.130
- net LVDS_TX3_N is gone; now on net VPA.: SLOT1.70
- net LVDS_TX3_P is gone; now on net E.: SLOT1.68
- net LVDS_TX4_P is gone; now on net RDY.: SLOT1.64
- net LVDS_TX5_P is gone; now on net PS2CLKIN: SLOT1.58
- net N6_IOR51A is gone; now on net _IRQ.: SLOT1.175
- net N7_IOR47B is gone; now on net _ABT.: SLOT1.177
- net N9_IOR36B is gone; now on net _NMI.: SLOT1.181
- net R9_IOR35A is gone; now on net _CSFLASH: SLOT1.183
- net VBUS is gone; now on net VCC: J8.7, J9.7
- net _WE is gone; now on net RW: U11.2 (DIR)
- net +3V3: now also J3.4 (VDD), R3.1, R4.1, U12.8 (VCC)
- net A0: now also U1.10 (A8); no longer U3.4 (A2)
- net A1: now also U1.9 (A7); no longer U3.6 (A4)
- net A10: now also U3.8 (A6); no longer U1.9 (A7)
- net A11: now also U3.7 (A5); no longer U1.10 (A8)
- net A12: now also U3.6 (A4); no longer U3.9 (A7)
- net A13: now also U3.5 (A3); no longer U3.7 (A5)
- net A13_IOR32A_READY: no longer SLOT1.98
- net A14: now also U3.4 (A2); no longer U3.5 (A3)
- net A2: now also U1.8 (A6); no longer U3.8 (A6)
- net A3: now also U1.7 (A5); no longer U3.10 (A8)
- net A4: now also U1.6 (A4); no longer U1.3 (A1)
- net A5: now also U1.5 (A3); no longer U1.4 (A2)
- net A6: now also U1.4 (A2); no longer U1.5 (A3)
- net A7: now also U1.3 (A1); no longer U1.6 (A4)
- net A8: now also U3.10 (A8); no longer U1.7 (A5)
- net A9: now also U3.9 (A7); no longer U1.8 (A6)
- net A_0: now also RN2.1 (R1.1); no longer RN4.3 (R3.1)
- net A_1: now also RN2.2 (R2.1); no longer RN4.1 (R1.1)
- net A_10: now also RN5.3 (R3.1); no longer RN2.2 (R2.1)
- net A_11: now also RN5.4 (R4.1); no longer RN2.1 (R1.1)
- net A_12: now also RN4.1 (R1.1); no longer RN5.2 (R2.1)
- net A_13: now also RN4.2 (R2.1); no longer RN5.4 (R4.1)
- net A_14: now also RN4.3 (R3.1); no longer RN4.2 (R2.1)
- net A_2: now also RN2.3 (R3.1); no longer RN5.3 (R3.1)
- net A_3: now also RN2.4 (R4.1); no longer RN5.1 (R1.1)
- net A_4: now also RN1.1 (R1.1); no longer RN1.4 (R4.1)
- net A_5: now also RN1.2 (R2.1); no longer RN1.3 (R3.1)
- net A_6: now also RN1.3 (R3.1); no longer RN1.2 (R2.1)
- net A_7: now also RN1.4 (R4.1); no longer RN1.1 (R1.1)
- net A_8: now also RN5.1 (R1.1); no longer RN2.4 (R4.1)
- net A_9: now also RN5.2 (R2.1); no longer RN2.3 (R3.1)
- net CA1: now also J6.11 (Pin_11), U24.5 (IN_5)
- net CA2: now also J6.12 (Pin_12), U24.6 (IN_6)
- net CB1: now also U25.7 (IN_7)
- net CB2: now also U25.6 (IN_6)
- net DATADIR: no longer RN3.8 (R1.2), U4.2 (DIR)
- net E: now also U7.3; no longer U7.13
- net GND: now also C3.2, D1.2 (A), J1.8 (Pin_8), J3.3 (VSS), J3.6 (VSS), J3.SH (SHELL), J6.2 (Pin_2), R1.1, SW1.3, SW1.4, U12.4 (GND), U24.1 (IN_1), U24.2 (IN_2), U24.3 (IN_3), U24.4 (IN_4), U24.8 (V-), U25.1 (IN_1), U25.2 (IN_2), U25.3 (IN_3), U25.4 (IN_4), U25.8 (V-); no longer U8.9
- net MISO: now also SLOT1.180, J3.7 (DAT0), U12.2 (DO/IO_{1})
- net MOSI: now also SLOT1.186, J3.2 (CMD), U12.5 (DI/IO_{0})
- net PA0: now also J6.3 (Pin_3), U24.15 (IN_14)
- net PA1: now also J6.4 (Pin_4), U24.14 (IN_13)
- net PA2: now also J6.5 (Pin_5), U24.13 (IN_12)
- net PA3: now also J6.6 (Pin_6), U24.12 (IN_11)
- net PA4: now also J6.7 (Pin_7), U24.11 (IN_10)
- net PA5: now also J6.8 (Pin_8), U24.10 (IN_9)
- net PA6: now also J6.9 (Pin_9), U24.9 (IN_8)
- net PA7: now also J6.10 (Pin_10), U24.7 (IN_7)
- net PB0: now also U25.15 (IN_14)
- net PB1: now also U25.14 (IN_13)
- net PB2: now also U25.13 (IN_12)
- net PB3: now also U25.12 (IN_11)
- net PB4: now also U25.11 (IN_10)
- net PB5: now also U25.10 (IN_9)
- net PB6: now also U25.9 (IN_8)
- net PB7: now also U25.5 (IN_5)
- net PS2DAT: now also U8.1, U8.4; no longer U8.10, U8.13
- net PSCLK: now also U8.10, U8.13; no longer U8.1, U8.4
- net RDY.: no longer U2.21 (B1)
- net SCK: now also SLOT1.182, J3.5 (CLK), U12.6 (CLK)
- net VCC: now also U1.2 (DIR), U3.2 (DIR), U6.2 (DIR), C3.1, D1.1 (K), F1.2, J1.1 (Pin_1), J6.1 (Pin_1), RN9.1 (R1.1), RN9.2 (R2.1), RN9.3 (R3.1), RN9.4 (R4.1), U24.16 (V+), U25.16 (V+); no longer J4.2 (Pin_2)
- net _816: now also U7.4, J1.6 (Pin_6); no longer U7.12
- net _ABT: now also RN8.7 (R2.2), J1.4 (Pin_4); no longer RN8.6 (R3.2)
- net _CESD: now also J3.1 (CD/DAT3)
- net _IRQ: now also RN8.6 (R3.2), U7.2, J1.3 (Pin_3); no longer RN8.7 (R2.2), U8.6
- net _NMI: now also J1.2 (Pin_2)
- net _RESET: now also RN8.8 (R1.2), U5.34 (BE), U7.12, U8.6, J1.5 (Pin_5); no longer U7.4
- net _RESET.: now also SLOT1.176, U13.7 (~{HOLD}/~{RESET}/IO_{3}), U7.13, U12.7 (~{HOLD}/~{RESET}/IO_{3}); no longer U7.3
- net _WPFLASH: now also R4.2, SW1.1
- net at U2.2 (DIR): now also R1.2
- net at U8.8: now also U8.5, RN9.6 (R3.2)
- net AVDD: no longer names the net of C1.1
- net AVDD: now also U8.9, R2.1, RN9.5 (R4.2)
- net B10_IOR31B_~{RECFG}: no longer names the net of SLOT1.96
- removed net BE: RN8.8 (R1.2), U5.34 (BE), U7.2
- net BE. renamed _IRQVIA
- net _IRQVIA: now also U10.17 (~{IRQ})
- net C7_IOL40B_1V5 renamed SW3
- net D10_IOL17A renamed PS2CLKIN
- net PS2CLKIN: now also RN10.7 (R2.2); no longer SLOT1.182
- net D11_IOL22A renamed PS2DATIN
- net PS2DATIN: now also RN10.8 (R1.2); no longer SLOT1.180
- net D7_IOL53B_1V5 renamed SW4
- removed net E10_IOL17B: RN10.7 (R2.2), SLOT1.186, U8.12
- net E8_IOL45B_1V5 renamed SW2
- net E9_IOL38B_1V5 renamed SW1
- removed net F10_IOL11A: RN10.8 (R1.2), SLOT1.176, U8.2
- net F14_IOT9A renamed D6.
- net F16_IOT9B renamed D7.
- net G14_IOT13B renamed D2.
- net G15_IOT13A renamed D3.
- net LVDS_IOR11_N renamed RW.
- net LVDS_IOR20_N renamed PHI2.
- net LVDS_IOR20_P renamed _CE_RAM1
- net LVDS_IOR40_P renamed _CSFLASH2
- net _CSFLASH2: now also U12.1 (~{CS})
- net LVDS_IOT18_P renamed A16
- net LVDS_IOT22_N renamed D5.
- net LVDS_IOT22_P renamed D4.
- net LVDS_IOT32_N renamed UD3_N
- net LVDS_IOT32_P renamed UD3_P
- net LVDS_IOT36_N renamed A18
- net LVDS_IOT36_P renamed A17
- net LVDS_IOT38_N renamed A20
- net LVDS_IOT38_P renamed A19
- net LVDS_IOT8_N renamed D1.
- net LVDS_IOT8_P renamed D0.
- net LVDS_RX1_P renamed PS2DATOUT
- net PS2DATOUT: now also U8.2
- net LVDS_RX2_N renamed B_TMDSC_N
- net LVDS_RX2_P renamed B_TMDSC_P
- net LVDS_RX3_N renamed B_TMDS0_N
- net LVDS_RX3_P renamed B_TMDS0_P
- net LVDS_RX4_N renamed B_TMDS1_P
- net LVDS_RX4_P renamed B_TMDS1_N
- net LVDS_RX5_N renamed B_TMDS2_P
- net LVDS_RX5_P renamed B_TMDS2_N
- net LVDS_TX4_N renamed _CE_RAM2
- net LVDS_TX5_N renamed PS2CLKOUT
- net PS2CLKOUT: now also U8.12
- net T4_IOB45B_1V5 renamed CARD_WP
- net CARD_WP: now also J3.11 (WRITE_PROTECT)
- net T5_IOB54B_1V5 renamed CARD_DET
- net CARD_DET: now also J3.10 (CARD_DETECT)
- removed net _IRQ.2: U10.17 (~{IRQ}), U8.5
- new net: F1.1, J4.2 (Pin_2)
- new net: J1.7 (Pin_7), R2.2
- new net DATADIR5V: RN3.8 (R1.2), U4.2 (DIR)
- new net _WPFLASH2: R3.2, SW1.2, U12.3 (~{WP}/IO_{2})
- no-connect marks 66 -> 56
Other:
- added sheet Audio - Video (C128_Audio.kicad_sch)
- added sheet Decoupling (C816_Decoupling.kicad_sch)
- added sheet ESP (C816_ESP.kicad_sch)
- added sheet SRAM 2MBx8 10nS (3V3_SRAM_2Mx8.kicad_sch)
- added sheet USB (C816_usb.kicad_sch)
- note added: "A13_IOR32A_READY"
- note added: "B10_IOR31B_~{RECFG}"
- note added: "ESP"
- note added: "F14_IOT9A"
- note added: "F16_IOT9B"
- note added: "G14_IOT13B"
- note added: "G15_IOT13A"
- note added: "LVDS_IOR20_N"
- note added: "LVDS_IOT22_N"
- note added: "LVDS_IOT22_P"
- note added: "LVDS_IOT40_P"
- note added: "LVDS_IOT8_N"
- note added: "LVDS_IOT8_P"
- note removed: "A16"
- note removed: "A17"
- note removed: "A18"
- note removed: "A19"
- note removed: "A20"
- note removed: "AUDIO"
- note removed: "ESD PROTECTION"
- note removed: "ESP32-C5 mini"
- note removed: "PS/2 CLK 3V3 IN"
- note removed: "PS/2 CLK 3V3 OUT"
- note removed: "PS/2 DAT 3V3 IN"
- note removed: "PS/2 DAT 3V3 OUT"
- note removed: "PULLUP IOPORTS"
- note removed: "SNES0/1"
- note removed: "SNES2/3"
- note removed: "USB SERIAL"
- note removed: "_CE1"
- note removed: "_RE"
- moved on the sheet: C2, RN10, RN8, U13, U8C, U8D
